Commit message: [feat]:初步实现机械臂移动到固定方块上方并下降、闭合夹爪的逻辑，但目前对于夹爪仅是位置调节，无法夹起方块，下一步应该加入力控制器，让夹爪对方块施加持续力，以夹起方块

File: src/robot_description/urdf/base.urdf.xacro (robot description, xacro)
@@ -103,5 +103,5 @@
             <origin xyz="0 -0.8 0" rpy="0 0 0"/>
             <axis xyz="0 0 1"/>
-            <limit effort="10" velocity="0.1" lower="-0.05" upper="0.0"/>
+            <limit effort="10" velocity="0.1" lower="-0.8" upper="0.0"/>
             <dynamics damping="0.1" friction="0.05"/>
         </joint>
@@ -136,6 +136,6 @@
             <origin xyz="0 -0.04 -0.23" rpy="0 0 0"/>
             <axis xyz="0 1 0"/>
-            <limit effort="5" velocity="0.05" lower="0.0" upper="0.02"/>
-            <dynamics damping="0.1" friction="0.01"/>
+            <limit effort="20" velocity="0.05" lower="0.0" upper="0.02"/>
+            <dynamics damping="0.5" friction="0.1"/>
         </joint>
         <link name="finger1">
@@ -163,4 +163,8 @@
         <gazebo reference="finger1">
             <material>Gazebo/Black</material>
+            <mu1 value="20.0" />
+            <mu2 value="20.0" />
+            <kp value="1000000000.0" />
+            <kd value="1.0" />
         </gazebo>
         <joint name="finger2_joint" type="prismatic">
@@ -196,4 +200,8 @@
         <gazebo reference="finger2">
             <material>Gazebo/Black</material>
+            <mu1 value="20.0" />
+            <mu2 value="20.0" />
+            <kp value="1000000000.0" />
+            <kd value="1.0" />
         </gazebo>
         <joint name="finger3_joint" type="prismatic">
@@ -229,4 +237,8 @@
         <gazebo reference="finger3">
             <material>Gazebo/Black</material>
+            <mu1 value="20.0" />
+            <mu2 value="20.0" />
+            <kp value="1000000000.0" />
+            <kd value="1.0" />
         </gazebo>
         <joint name="finger4_joint" type="prismatic">
@@ -262,4 +274,8 @@
         <gazebo reference="finger4">
             <material>Gazebo/Black</material>
+            <mu1 value="20.0" />
+            <mu2 value="20.0" />
+            <kp value="1000000000.0" />
+            <kd value="1.0" />
         </gazebo>
     </xacro:macro>

Commit message: [fix]:优化gazebo下的机械臂显示效果

File: src/robot_description/urdf/base.urdf.xacro (robot description, xacro)
@@ -19,6 +19,6 @@
                     <cylinder length="0.4" radius="0.1"/>
                 </geometry>
-                <material name="space_gray">
-                    <color rgba="0.3 0.3 0.35 1.0"/>
+                <material name="dark_gray">
+                    <color rgba="0.4 0.4 0.4 1.0"/>
                 </material>
             </visual>
@@ -30,5 +30,5 @@
         </link>
         <gazebo reference="base_link">
-            <material>Gazebo/DarkGrey</material>
+            <material>Gazebo/White</material>
         </gazebo>
         <joint name="rotation1" type="revolute">
@@ -52,6 +52,6 @@
                     <box size="0.1 1.1 0.1"/>
                 </geometry>
-                <material name="silver">
-                    <color rgba="0.88 0.88 0.90 1.0"/>
+                <material name="dark_gray">
+                    <color rgba="0.4 0.4 0.4 1.0"/>
                 </material>
             </visual>
@@ -63,5 +63,5 @@
         </link>
         <gazebo reference="arm1">
-            <material>Gazebo/Black</material>
+            <material>Gazebo/White</material>
         </gazebo>
         <joint name="rotation2" type="revolute">
@@ -85,6 +85,6 @@
                     <box size="0.1 0.9 0.1"/>
                 </geometry>
-                <material name="silver2">
-                    <color rgba="0.88 0.88 0.90 1.0"/>
+                <material name="dark_gray">
+                    <color rgba="0.4 0.4 0.4 1.0"/>
                 </material>
             </visual>
@@ -96,5 +96,5 @@
         </link>
         <gazebo reference="arm2">
-            <material>Gazebo/Black</material>
+            <material>Gazebo/White</material>
         </gazebo>
         <joint name="gripper_joint" type="prismatic">
@@ -118,6 +118,6 @@
                     <cylinder length="0.2" radius="0.02"/>
                 </geometry>
-                <material name="matte_black">
-                    <color rgba="0.15 0.15 0.18 1.0"/>
+                <material name="dark_gray">
+                    <color rgba="0.4 0.4 0.4 1.0"/>
                 </material>
             </visual>
@@ -129,5 +129,5 @@
         </link>
         <gazebo reference="gripper_link">
-            <material>Gazebo/Black</material>
+            <material>Gazebo/White</material>
         </gazebo>
         <joint name="finger1_joint" type="prismatic">
@@ -151,6 +151,6 @@
                     <box size="0.02 0.01 0.02"/>
                 </geometry>
-                <material name="light_aluminum">
-                    <color rgba="0.92 0.92 0.94 1.0"/>
+                <material name="dark_gray">
+                    <color rgba="0.4 0.4 0.4 1.0"/>
                 </material>
             </visual>
@@ -162,5 +162,5 @@
         </link>
         <gazebo reference="finger1">
-            <material>Gazebo/Black</material>
+            <material>Gazebo/White</material>
             <mu1 value="20.0" />
             <mu2 value="20.0" />
@@ -188,6 +188,6 @@
                     <box size="0.01 0.02 0.02"/>
                 </geometry>
-                <material name="light_aluminum2">
-                    <color rgba="0.92 0.92 0.94 1.0"/>
+                <material name="dark_gray">
+                    <color rgba="0.4 0.4 0.4 1.0"/>
                 </material>
             </visual>
@@ -199,5 +199,5 @@
         </link>
         <gazebo reference="finger2">
-            <material>Gazebo/Black</material>
+            <material>Gazebo/White</material>
             <mu1 value="20.0" />
             <mu2 value="20.0" />
@@ -225,6 +225,6 @@
                     <box size="0.02 0.01 0.02"/>
                 </geometry>
-                <material name="light_aluminum3">
-                    <color rgba="0.92 0.92 0.94 1.0"/>
+                <material name="dark_gray">
+                    <color rgba="0.4 0.4 0.4 1.0"/>
                 </material>
             </visual>
@@ -236,5 +236,5 @@
         </link>
         <gazebo reference="finger3">
-            <material>Gazebo/Black</material>
+            <material>Gazebo/White</material>
             <mu1 value="20.0" />
             <mu2 value="20.0" />
@@ -262,6 +262,6 @@
                     <box size="0.01 0.02 0.02"/>
                 </geometry>
-                <material name="light_aluminum4">
-                    <color rgba="0.92 0.92 0.94 1.0"/>
+                <material name="dark_gray">
+                    <color rgba="0.4 0.4 0.4 1.0"/>
                 </material>
             </visual>
@@ -273,5 +273,5 @@
         </link>
         <gazebo reference="finger4">
-            <material>Gazebo/Black</material>
+            <material>Gazebo/White</material>
             <mu1 value="20.0" />
             <mu2 value="20.0" />

Commit message: [feat]:修改手指部分参数

File: src/robot_description/urdf/base.urdf.xacro (robot description, xacro)
@@ -173,6 +173,6 @@
             <origin xyz="0.04 0 -0.23" rpy="0 0 0"/>
             <axis xyz="1 0 0"/>
-            <limit effort="5" velocity="0.05" lower="-0.02" upper="0.0"/>
-            <dynamics damping="0.1" friction="0.01"/>
+            <limit effort="20" velocity="0.05" lower="-0.02" upper="0.0"/>
+            <dynamics damping="0.5" friction="0.1"/>
         </joint>
         <link name="finger2">
@@ -210,6 +210,6 @@
             <origin xyz="0 0.04 -0.23" rpy="0 0 0"/>
             <axis xyz="0 1 0"/>
-            <limit effort="5" velocity="0.05" lower="-0.02" upper="0.0"/>
-            <dynamics damping="0.1" friction="0.01"/>
+            <limit effort="20" velocity="0.05" lower="-0.02" upper="0.0"/>
+            <dynamics damping="0.5" friction="0.1"/>
         </joint>
         <link name="finger3">
@@ -247,6 +247,6 @@
             <origin xyz="-0.04 0 -0.23" rpy="0 0 0"/>
             <axis xyz="1 0 0"/>
-            <limit effort="5" velocity="0.05" lower="0.0" upper="0.02"/>
-            <dynamics damping="0.1" friction="0.01"/>
+            <limit effort="20" velocity="0.05" lower="0.0" upper="0.02"/>
+            <dynamics damping="0.5" friction="0.1"/>
         </joint>
         <link name="finger4">

Commit message: [fix]:小改参数，目前仍在探讨位控制实现夹取的可能性

File: src/robot_description/urdf/base.urdf.xacro (robot description, xacro)
@@ -136,9 +136,9 @@
             <origin xyz="0 -0.04 -0.23" rpy="0 0 0"/>
             <axis xyz="0 1 0"/>
-            <limit effort="20" velocity="0.05" lower="0.0" upper="0.02"/>
-            <dynamics damping="0.5" friction="0.1"/>
+            <limit effort="20" velocity="0.05" lower="0.0" upper="0.04"/>
+            <dynamics damping="0.1" friction="0.1"/>
         </joint>
         <link name="finger1">
-            <collision>
+            <collision name="finger1_collision">
                 <origin xyz="0 0 0" rpy="0 0 0"/>
                 <geometry>
@@ -173,9 +173,9 @@
             <origin xyz="0.04 0 -0.23" rpy="0 0 0"/>
             <axis xyz="1 0 0"/>
-            <limit effort="20" velocity="0.05" lower="-0.02" upper="0.0"/>
-            <dynamics damping="0.5" friction="0.1"/>
+            <limit effort="20" velocity="0.05" lower="-0.04" upper="0.0"/>
+            <dynamics damping="0.1" friction="0.1"/>
         </joint>
         <link name="finger2">
-            <collision>
+            <collision name="finger2_collision">
                 <origin xyz="0 0 0" rpy="0 0 0"/>
                 <geometry>
@@ -210,9 +210,9 @@
             <origin xyz="0 0.04 -0.23" rpy="0 0 0"/>
             <axis xyz="0 1 0"/>
-            <limit effort="20" velocity="0.05" lower="-0.02" upper="0.0"/>
-            <dynamics damping="0.5" friction="0.1"/>
+            <limit effort="20" velocity="0.05" lower="-0.04" upper="0.0"/>
+            <dynamics damping="0.1" friction="0.1"/>
         </joint>
         <link name="finger3">
-            <collision>
+            <collision name="finger3_collision">
                 <origin xyz="0 0 0" rpy="0 0 0"/>
                 <geometry>
@@ -247,9 +247,9 @@
             <origin xyz="-0.04 0 -0.23" rpy="0 0 0"/>
             <axis xyz="1 0 0"/>
-            <limit effort="20" velocity="0.05" lower="0.0" upper="0.02"/>
-            <dynamics damping="0.5" friction="0.1"/>
+            <limit effort="20" velocity="0.05" lower="0.0" upper="0.04"/>
+            <dynamics damping="0.1" friction="0.1"/>
         </joint>
         <link name="finger4">
-            <collision>
+            <collision name="finger4_collision">
                 <origin xyz="0 0 0" rpy="0 0 0"/>
                 <geometry>

File: src/robot_description/urdf/robot.ros2_control.xacro (robot description, xacro)
@@ -32,4 +32,5 @@
         <joint name="finger1_joint">
             <command_interface name="position"/>
+            <state_interface name="effort"/>
             <state_interface name="position"/>
             <state_interface name="velocity"/>
@@ -37,4 +38,5 @@
         <joint name="finger2_joint">
             <command_interface name="position"/>
+            <state_interface name="effort"/>
             <state_interface name="position"/>
             <state_interface name="velocity"/>
@@ -42,4 +44,5 @@
         <joint name="finger3_joint">
             <command_interface name="position"/>
+            <state_interface name="effort"/>
             <state_interface name="position"/>
             <state_interface name="velocity"/>
@@ -47,4 +50,5 @@
         <joint name="finger4_joint">
             <command_interface name="position"/>
+            <state_interface name="effort"/>
             <state_interface name="position"/>
             <state_interface name="velocity"/>
